File: binaryclock-kicad/binaryclock.kicad_pcb (KiCad board)
At the start: 2 copper layers, 100 x 80 mm, 19 parts, among them J1 Conn_01x03_Pin, J2 AVR-ISP-6, SW1 SW_Push, SW2 SW_Push, SW3 SW_Push, U1 ATmega48-20P, Y1 Crystal

Commit message: prettified pcb
Parts:
- added G***: LOGO, LOGO, F.Cu at (120.0, 70.0)
Routing:
- net +BATT: track 84.3 -> 77.1 mm
- net /MOSI/PCINT3: track 171.9 -> 165.2 mm, vias 4 -> 2
- net /SCK: track 64.6 -> 63.0 mm
Other:
- board text added: "(>_>)"
- board text added: "BINARY CLOCK Σ-EDITION"

Commit message: did some adjustments
Routing:
- net +BATT: track 77.1 -> 81.3 mm
Changed lines of the file:
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@@
 		(tenting front back)
 		(pcbplotparams
-			(layerselection 0x00000000_00000000_55555555_5755f5ff)
+			(layerselection 0x00000000_00000000_55555555_57555555)
 			(plot_on_all_layers_selection 0x00000000_00000000_00000000_00000000)
 			(disableapertmacros no)
@@
 			(outputformat 1)
 			(mirror no)
-			(drillshape 1)
+			(drillshape 0)
 			(scaleselection 1)
-			(outputdirectory "")
+			(outputdirectory "C:/Users/david/Downloads/")
 		)
 	)
@@
 	)
 	(segment
-		(start 132 64.5)
-		(end 120.25 52.75)
+		(start 117.5 52.632055)
+		(end 117.632055 52.632055)
 		(width 0.8)
 		(layer "F.Cu")
@@
 	)
 	(segment
-		(start 132 80.75)
-		(end 132 64.5)
+		(start 132 67)
+		(end 132 80.75)
+		(width 0.8)
+		(layer "F.Cu")
+		(net 2)
+	)
+	(segment
+		(start 117.632055 52.632055)
+		(end 132 67)
 		(width 0.8)
 		(layer "F.Cu")
@@
 	)
 	(via
-		(at 120.25 52.75)
+		(at 117.5 52.632055)
 		(size 2)
 		(drill 0.9)
@@
 	)
 	(segment
-		(start 125.25 52.749999)
-		(end 120.25 52.75)
+		(start 139 109.25)
+		(end 139.689 108.561)
 		(width 0.8)
 		(layer "B.Cu")
@@
 	)
 	(segment
-		(start 139 109.25)
-		(end 139.689 108.561)
+		(start 117.617944 52.749999)
+		(end 117.5 52.632055)
 		(width 0.8)
 		(layer "B.Cu")
@@
 	)
 	(segment
+		(start 125.25 52.749999)
+		(end 117.617944 52.749999)
+		(width 0.8)
+		(layer "B.Cu")
+		(net 2)
+	)
+	(segment
 		(start 141.16 85.84)
 		(end 141.736999 85.84)
@@
 	)
 	(segment
+		(start 132.79 111.79)
+		(end 139 111.79)
+		(width 0.8)
+		(layer "B.Cu")
+		(net 21)
+	)
+	(segment
 		(start 89.75 112.25)
 		(end 138.54 112.25)
@@
 	)
 	(segment
-		(start 124.25 103.25)
-		(end 132.79 111.79)
+		(start 138.54 112.25)
+		(end 139 111.79)
 		(width 0.8)
 		(layer "B.Cu")
@@
 	)
 	(segment
-		(start 138.54 112.25)
-		(end 139 111.79)
+		(start 124.25 103.25)
+		(end 132.79 111.79)
 		(width 0.8)
 		(layer "B.Cu")
@@
 		(width 0.8)
 		(layer "B.Cu")
-		(net 21)
-	)
-	(segment
-		(start 132.79 111.79)
-		(end 139 111.79)
-		(width 0.8)
-		(layer "B.Cu")
