File: binaryclock-kicad/binaryclock.kicad_pcb (KiCad board)
At the start: 2 copper layers, 100 x 80 mm, 20 parts, among them J1 Conn_01x03_Pin, J2 AVR-ISP-6, SW1 SW_Push, SW2 SW_Push, SW3 SW_Push, U1 ATmega48-20P, Y1 Crystal

Commit message: finished pcb
Parts:
- moved SW1 0.50 mm to (63.2, 112.2)
- moved SW3 0.50 mm to (85.8, 112.2)
Routing:
- net /MISO/PCINT4: track 114.9 -> 114.4 mm
Other:
- board text added: "DBG"
- board text added: "DISP"
- board text added: "SET"
- board text added: "↑"
- board text added: "↓"
- board text removed: "SW1"
- board text removed: "SW2"
- board text removed: "SW3"
Changed lines of the file:
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@@
 		(tenting front back)
 		(pcbplotparams
-			(layerselection 0x00000000_00000000_55555555_57555555)
+			(layerselection 0x00000000_00000000_55555555_55555555)
 			(plot_on_all_layers_selection 0x00000000_00000000_00000000_00000000)
 			(disableapertmacros no)
@@
 			(drillshape 0)
 			(scaleselection 1)
-			(outputdirectory "C:/Users/david/Downloads/")
+			(outputdirectory "../fabrication-outputs/")
 		)
 	)
@@
 	(footprint "Button_Switch_THT:SW_PUSH_6mm"
 		(layer "F.Cu")
-		(at 63.75 112.25 90)
+		(at 63.25 112.25 90)
 		(descr "Generic 6mm SW tactile push button")
 		(tags "tact sw push 6mm")
@@
 	(footprint "Button_Switch_THT:SW_PUSH_6mm"
 		(layer "F.Cu")
-		(at 85.25 112.25 90)
+		(at 85.75 112.25 90)
 		(descr "Generic 6mm SW tactile push button")
 		(tags "tact sw push 6mm")
@@
 		)
 	)
-	(gr_text "SW1"
-		(at 61.75 103.25 0)
+	(gr_text "DISP"
+		(at 61 117.5 0)
 		(layer "F.Cu" knockout)
 		(effects
@@
 		)
 	)
-	(gr_text "SW2"
-		(at 72.5 103.25 0)
+	(gr_text "SET"
+		(at 73 117.5 0)
 		(layer "F.Cu" knockout)
 		(effects
@@
 		)
 	)
-	(gr_text "SW3"
-		(at 83.25 103.25 0)
+	(gr_text "DBG"
+		(at 83.75 117.5 0)
 		(layer "F.Cu" knockout)
 		(effects
@@
 		)
 	)
+	(gr_text "↑"
+		(at 80 112.25 0)
+		(layer "F.Cu" knockout)
+		(effects
+			(font
+				(size 7 3)
+				(thickness 0.6)
+				(bold yes)
+			)
+			(justify left bottom)
+		)
+	)
 	(gr_text "MINUTES"
 		(at 62.75 79.5 0)
@@
 		)
 	)
+	(gr_text "↓"
+		(at 91.5 112.25 0)
+		(layer "F.Cu" knockout)
+		(effects
+			(font
+				(size 7 3)
+				(thickness 0.6)
+				(bold yes)
+			)
+			(justify left bottom)
+		)
+	)
 	(gr_text "BINARY\nCLOCK\nΣ-EDITION"
-		(at 108.5 113 0)
+		(at 109.666661 111.796146 0)
 		(layer "F.Cu" knockout)
 		(effects
@@
 	)
 	(segment
-		(start 132.79 111.79)
+		(start 138.54 112.25)
 		(end 139 111.79)
 		(width 0.8)
@@
 	)
 	(segment
-		(start 89.75 112.25)
-		(end 138.54 112.25)
-		(width 0.8)
-		(layer "B.Cu")
-		(net 21)
-	)
-	(segment
-		(start 124.25 78)
-		(end 126.57 75.68)
+		(start 132.79 111.79)
+		(end 139 111.79)
 		(width 0.8)
 		(layer "B.Cu")
@@
 	)
 	(segment
-		(start 89.75 105.75)
-		(end 89.75 112.25)
+		(start 90.25 105.75)
+		(end 90.25 112.25)
 		(width 0.8)
 		(layer "B.Cu")
@@
 	)
 	(segment
-		(start 138.54 112.25)
-		(end 139 111.79)
+		(start 124.25 78)
+		(end 126.57 75.68)
 		(width 0.8)
 		(layer "B.Cu")
@@
 	)
 	(segment
+		(start 90.25 112.25)
+		(end 138.54 112.25)
+		(width 0.8)
+		(layer "B.Cu")
+		(net 21)
+	)
+	(segment
 		(start 150.499 116.751)
 		(end 152 115.25)
@@
 	)
 	(segment
-		(start 68.25 105.75)
-		(end 68.25 112.25)
-		(width 0.8)
-		(layer "B.Cu")
-		(net 22)
-	)
-	(segment
-		(start 72.751 116.751)
-		(end 68.25 112.25)
-		(width 0.8)
-		(layer "B.Cu")
-		(net 22)
-	)
-	(segment
-		(start 117.249 116.751)
-		(end 72.751 116.751)
+		(start 67.75 112.25)
+		(end 72.25 116.75)
 		(width 0.8)
 		(layer "B.Cu")
@@
 	)
 	(segment
-		(start 117.25 116.75)
-		(end 117.249 116.751)
+		(start 72.25 116.75)
+		(end 120.25 116.75)
 		(width 0.8)
 		(layer "B.Cu")
@@
 	)
 	(segment
-		(start 120.25 116.75)
-		(end 117.25 116.75)
+		(start 67.75 105.75)
+		(end 67.75 112.25)
 		(width 0.8)
 		(layer "B.Cu")

Commit message: TRUE FINAL PCB VERSION
Parts:
- Y1: footprint Crystal:Crystal_Round_D2.0mm_Vertical -> Connector_PinHeader_2.54mm:PinHeader_1x02_P2.54mm_Vertical
- moved Y1 2.29 mm to (146.4, 81.8), turned to 180 degrees
- moved D4 1.66 mm to (80.9, 65.4)
- moved D5 1.66 mm to (86.7, 65.4)
- moved D9 1.66 mm to (80.2, 83.9)
- moved J1 1.66 mm to (149.9, 94.4)
- moved J2 1.66 mm to (137.7, 112.8)
- moved U1 1.66 mm to (142.5, 102.1)
- moved SW1 1.66 mm to (61.9, 113.2)
- moved BT1 1.66 mm to (123.9, 53.7)
- moved D1 1.66 mm to (63.6, 65.4)
- moved D10 1.66 mm to (85.9, 83.9)
- moved D11 1.66 mm to (91.7, 83.9)
- moved D2 1.66 mm to (69.4, 65.4)
- moved D3 1.66 mm to (75.2, 65.4)
- moved D6 1.66 mm to (63.0, 83.9)
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Routing:
- net /MISO/PCINT4: track 114.4 -> 107.7 mm
- net /MOSI/PCINT3: track 165.2 -> 170.2 mm
- net /PC5: track 77.2 -> 73.8 mm
- net /PD3: track 129.1 -> 130.9 mm
- net /SCK: track 63.0 -> 61.8 mm
- net /PD4: track 119.1 -> 120.3 mm
- net /PC4: track 78.8 -> 77.8 mm
- net /PC3: track 80.7 -> 79.7 mm
- net /TOSC1: track 4.60 -> 3.90 mm
